Commit message: Aligned mesh visulaization

File: src/agriscout_description/urdf/agriscout.urdf.xacro (robot description, xacro)
@@ -4,5 +4,5 @@
     <link name="base_link">
         <visual>
-            <origin xyz="-0.09 0.13 0" rpy="1.57 0 0"/>
+            <origin xyz="-0.11 -0.1 0" rpy="1.57 0 1.57"/>
             <geometry>
                 <mesh filename="package://agriscout_description/meshes/chassis.STL" scale="0.001 0.001 0.001"/>
@@ -30,5 +30,5 @@
     <link name="left_track">
         <visual>
-            <origin xyz="-0.09 0 0" rpy="1.57 0 0"/>
+            <origin xyz="-0.15 -0.04 0" rpy="1.57 0 1.57"/>
             <geometry>
                 <mesh filename="package://agriscout_description/meshes/track.STL" scale="0.001 0.001 0.001"/>
@@ -46,5 +46,5 @@
     <link name="right_track">
         <visual>
-            <origin xyz="0.07 0.24 0" rpy="1.57 0 0"/>
+            <origin xyz="-0.15 0.01 0" rpy="1.57 0 1.57"/>
             <geometry>
                 <mesh filename="package://agriscout_description/meshes/track.STL" scale="0.001 0.001 0.001"/>

Commit message: Created a four wheel drive joint system

File: src/agriscout_description/urdf/agriscout.urdf.xacro (robot description, xacro)
@@ -4,5 +4,5 @@
     <link name="base_link">
         <visual>
-            <origin xyz="-0.11 -0.1 0" rpy="1.57 0 1.57"/>
+            <origin xyz="-0.11 -0.1 -0.03" rpy="1.57 0 1.57"/>
             <geometry>
                 <mesh filename="package://agriscout_description/meshes/chassis.STL" scale="0.001 0.001 0.001"/>
@@ -28,7 +28,7 @@
         <origin xyz="0 0 0" rpy="0 0 0"/>
     </joint>
-    <link name="left_track">
+    <link name="left_track_visual">
         <visual>
-            <origin xyz="-0.15 -0.04 0" rpy="1.57 0 1.57"/>
+            <origin xyz="-0.15 -0.04 -0.03" rpy="1.57 0 1.57"/>
             <geometry>
                 <mesh filename="package://agriscout_description/meshes/track.STL" scale="0.001 0.001 0.001"/>
@@ -38,13 +38,13 @@
             </material>
         </visual>
-        <collision>
-            <geometry>
-                <box size="0.25 0.05 0.1"/>
-            </geometry>
-        </collision>
-    </link>
-    <link name="right_track">
+        </link>
+    <joint name="left_track_visual_joint" type="fixed">
+        <parent link="base_link"/>
+        <child link="left_track_visual"/>
+        <origin xyz="0 0.12 0.04" rpy="0 0 0"/>
+    </joint>
+    <link name="right_track_visual">
         <visual>
-            <origin xyz="-0.15 0.01 0" rpy="1.57 0 1.57"/>
+            <origin xyz="-0.15 0.01 -0.03" rpy="1.57 0 1.57"/>
             <geometry>
                 <mesh filename="package://agriscout_description/meshes/track.STL" scale="0.001 0.001 0.001"/>
@@ -52,21 +52,67 @@
             <material name="black"/>
         </visual>
+    </link>
+    <joint name="right_track_visual_joint" type="fixed">
+        <parent link="base_link"/>
+        <child link="right_track_visual"/>
+        <origin xyz="0 -0.12 0.04" rpy="0 0 0"/>
+    </joint>
+    <link name="left_rear_wheel">
         <collision>
+            <origin xyz="0 0 0" rpy="1.57 0 0"/>
             <geometry>
-                <box size="0.25 0.05 0.1"/>
+                <cylinder length="0.04" radius="0.04"/>
             </geometry>
         </collision>
     </link>
-    <joint name="left_track_joint" type="fixed">
+    <joint name="left_rear_joint" type="continuous">
         <parent link="base_link"/>
-        <child link="left_track"/>
-        <origin xyz="0 0.12 0.04" rpy="0 0 0"/>
+        <child link="left_rear_wheel"/>
+        <origin xyz="-0.09 0.12 0.04" rpy="0 0 0"/>
+        <axis xyz="0 1 0"/>
     </joint>
-    <joint name="right_track_joint" type="fixed">
+    <link name="left_front_wheel">
+        <collision>
+            <origin xyz="0 0 0" rpy="1.57 0 0"/>
+            <geometry>
+                <cylinder length="0.04" radius="0.04"/>
+            </geometry>
+        </collision>
+    </link>
+    <joint name="left_front_joint" type="continuous">
         <parent link="base_link"/>
-        <child link="right_track"/>
-        <origin xyz="0 -0.12 0.04" rpy="0 0 0"/>
+        <child link="left_front_wheel"/>
+        <origin xyz="0.09 0.12 0.04" rpy="0 0 0"/>
+        <axis xyz="0 1 0"/>
     </joint>
-   <link name="camera_link">
+    <link name="right_rear_wheel">
+        <collision>
+            <origin xyz="0 0 0" rpy="1.57 0 0"/>
+            <geometry>
+                <cylinder length="0.04" radius="0.04"/>
+            </geometry>
+        </collision>
+    </link>
+    <joint name="right_rear_joint" type="continuous">
+        <parent link="base_link"/>
+        <child link="right_rear_wheel"/>
+        <origin xyz="-0.09 -0.12 0.04" rpy="0 0 0"/>
+        <axis xyz="0 1 0"/>
+    </joint>
+    <link name="right_front_wheel">
+        <collision>
+            <origin xyz="0 0 0" rpy="1.57 0 0"/>
+            <geometry>
+                <cylinder length="0.04" radius="0.04"/>
+            </geometry>
+        </collision>
+    </link>
+    <joint name="right_front_joint" type="continuous">
+        <parent link="base_link"/>
+        <child link="right_front_wheel"/>
+        <origin xyz="0.09 -0.12 0.04" rpy="0 0 0"/>
+        <axis xyz="0 1 0"/>
+    </joint>
+    <link name="camera_link">
         <visual>
             <geometry>

Commit message: Finally aligned vision geometry with collision geometry in the visualization

File: src/agriscout_description/urdf/agriscout.urdf.xacro (robot description, xacro)
@@ -4,5 +4,5 @@
     <link name="base_link">
         <visual>
-            <origin xyz="-0.11 -0.1 -0.03" rpy="1.57 0 1.57"/>
+            <origin xyz="-0.11 -0.1 -0.05" rpy="1.57 0 1.57"/>
             <geometry>
                 <mesh filename="package://agriscout_description/meshes/chassis.STL" scale="0.001 0.001 0.001"/>
@@ -13,7 +13,7 @@
         </visual>
         <collision>
-            <origin xyz="0 0 0.05" rpy="0 0 0"/>
+            <origin xyz="0 -0.0135 0.03" rpy="0 0 0"/>
             <geometry>
-                <box size="0.24 0.18 0.08"/>
+                <box size="0.22 0.14 0.06"/>
             </geometry>
         </collision>
@@ -28,9 +28,9 @@
         <origin xyz="0 0 0" rpy="0 0 0"/>
     </joint>
-    <link name="left_track_visual">
+    <link name="left_rear_wheel">
         <visual>
-            <origin xyz="-0.15 -0.04 -0.03" rpy="1.57 0 1.57"/>
+            <origin xyz="0 0 0" rpy="1.57 0 0"/>
             <geometry>
-                <mesh filename="package://agriscout_description/meshes/track.STL" scale="0.001 0.001 0.001"/>
+                <cylinder length="0.02" radius="0.035"/>
             </geometry>
             <material name="black">
@@ -38,78 +38,94 @@
             </material>
         </visual>
-        </link>
-    <joint name="left_track_visual_joint" type="fixed">
-        <parent link="base_link"/>
-        <child link="left_track_visual"/>
-        <origin xyz="0 0.12 0.04" rpy="0 0 0"/>
-    </joint>
-    <link name="right_track_visual">
-        <visual>
-            <origin xyz="-0.15 0.01 -0.03" rpy="1.57 0 1.57"/>
-            <geometry>
-                <mesh filename="package://agriscout_description/meshes/track.STL" scale="0.001 0.001 0.001"/>
-            </geometry>
-            <material name="black"/>
-        </visual>
-    </link>
-    <joint name="right_track_visual_joint" type="fixed">
-        <parent link="base_link"/>
-        <child link="right_track_visual"/>
-        <origin xyz="0 -0.12 0.04" rpy="0 0 0"/>
-    </joint>
-    <link name="left_rear_wheel">
         <collision>
             <origin xyz="0 0 0" rpy="1.57 0 0"/>
             <geometry>
-                <cylinder length="0.04" radius="0.04"/>
+                <cylinder length="0.02" radius="0.035"/>
             </geometry>
         </collision>
+        <inertial>
+            <mass value="0.2"/>
+            <inertia ixx="0.001" ixy="0" ixz="0" iyy="0.001" iyz="0" izz="0.001"/>
+        </inertial>
     </link>
     <joint name="left_rear_joint" type="continuous">
         <parent link="base_link"/>
         <child link="left_rear_wheel"/>
-        <origin xyz="-0.09 0.12 0.04" rpy="0 0 0"/>
+        <origin xyz="-0.035 0.065 0.03" rpy="0 0 0"/>
         <axis xyz="0 1 0"/>
     </joint>
     <link name="left_front_wheel">
+        <visual>
+            <origin xyz="0 0 0" rpy="1.57 0 0"/>
+            <geometry>
+                <cylinder length="0.02" radius="0.035"/>
+            </geometry>
+            <material name="black"/>
+        </visual>
         <collision>
             <origin xyz="0 0 0" rpy="1.57 0 0"/>
             <geometry>
-                <cylinder length="0.04" radius="0.04"/>
+                <cylinder length="0.02" radius="0.035"/>
             </geometry>
         </collision>
+        <inertial>
+            <mass value="0.2"/>
+            <inertia ixx="0.001" ixy="0" ixz="0" iyy="0.001" iyz="0" izz="0.001"/>
+        </inertial>
     </link>
     <joint name="left_front_joint" type="continuous">
         <parent link="base_link"/>
         <child link="left_front_wheel"/>
-        <origin xyz="0.09 0.12 0.04" rpy="0 0 0"/>
+        <origin xyz="0.073 0.065 0.03" rpy="0 0 0"/>
         <axis xyz="0 1 0"/>
     </joint>
     <link name="right_rear_wheel">
+        <visual>
+            <origin xyz="0 0 0" rpy="1.57 0 0"/>
+            <geometry>
+                <cylinder length="0.02" radius="0.035"/>
+            </geometry>
+            <material name="black"/>
+        </visual>
         <collision>
             <origin xyz="0 0 0" rpy="1.57 0 0"/>
             <geometry>
-                <cylinder length="0.04" radius="0.04"/>
+                <cylinder length="0.02" radius="0.035"/>
             </geometry>
         </collision>
+        <inertial>
+            <mass value="0.2"/>
+            <inertia ixx="0.001" ixy="0" ixz="0" iyy="0.001" iyz="0" izz="0.001"/>
+        </inertial>
     </link>
     <joint name="right_rear_joint" type="continuous">
         <parent link="base_link"/>
         <child link="right_rear_wheel"/>
-        <origin xyz="-0.09 -0.12 0.04" rpy="0 0 0"/>
+        <origin xyz="-0.035 -0.09 0.03" rpy="0 0 0"/>
         <axis xyz="0 1 0"/>
     </joint>
     <link name="right_front_wheel">
+        <visual>
+            <origin xyz="0 0 0" rpy="1.57 0 0"/>
+            <geometry>
+                <cylinder length="0.02" radius="0.035"/>
+            </geometry>
+            <material name="black"/>
+        </visual>
         <collision>
             <origin xyz="0 0 0" rpy="1.57 0 0"/>
             <geometry>
-                <cylinder length="0.04" radius="0.04"/>
+                <cylinder length="0.02" radius="0.035"/>
             </geometry>
         </collision>
+        <inertial>
+            <mass value="0.2"/>
+            <inertia ixx="0.001" ixy="0" ixz="0" iyy="0.001" iyz="0" izz="0.001"/>
+        </inertial>
     </link>
     <joint name="right_front_joint" type="continuous">
         <parent link="base_link"/>
         <child link="right_front_wheel"/>
-        <origin xyz="0.09 -0.12 0.04" rpy="0 0 0"/>
+        <origin xyz="0.073 -0.09 0.03" rpy="0 0 0"/>
         <axis xyz="0 1 0"/>
     </joint>
@@ -122,9 +138,14 @@
             </material>
         </visual>
+        <collision>
+             <geometry>
+                <box size="0.025 0.025 0.025"/>
+            </geometry>
+        </collision>
     </link>
     <joint name="camera_joint" type="fixed">
         <parent link="base_link"/>
         <child link="camera_link"/>
-        <origin xyz="0.12 0 0.08" rpy="0 0 0"/>
+        <origin xyz="0.12 -0.0135 0.08" rpy="0 0 0"/>
     </joint>
     <link name="camera_optical_link"/>
@@ -147,5 +168,5 @@
         <parent link="base_link"/>
         <child link="imu_link"/>
-        <origin xyz="0 0 0.06" rpy="0 0 0"/>
+        <origin xyz="0 -0.0135 0.06" rpy="0 0 0"/>
     </joint>
 </robot>

Commit message: Refined The entire Workspace and Created the First Gazebo Simulation

File: src/agriscout_description/urdf/agriscout.urdf.xacro (robot description, xacro)
@@ -1,4 +1,5 @@
 <?xml version="1.0"?>
 <robot xmlns:xacro="http://www.ros.org/wiki/xacro" name="agriscout">
+<xacro:include filename="$(find agriscout_description)/urdf/gazebo.xacro" />
     <link name="base_footprint"/>
     <link name="base_link">
@@ -170,3 +171,20 @@
         <origin xyz="0 -0.0135 0.06" rpy="0 0 0"/>
     </joint>
+    <link name="lidar_link">
+        <visual>
+            <geometry>
+                <cylinder length="0.04" radius="0.035"/>
+            </geometry>
+            <material name="black"/>
+        </visual>
+        <collision>
+            <geometry>
+                <cylinder length="0.04" radius="0.035"/>
+            </geometry>
+        </collision>
+    </link>
+    <joint name="lidar_joint" type="fixed">
+        <parent link="base_link"/>
+        <child link="lidar_link"/>
+        <origin xyz="0 0 0.1" rpy="0 0 0"/> </joint>
 </robot>

Commit message: Debugged the Motor Controlled manager (TwistStamped) and implemented the agriscout_vision pkg

File: src/agriscout_description/urdf/agriscout.urdf.xacro (robot description, xacro)
@@ -16,5 +16,5 @@
             <origin xyz="0 -0.0135 0.03" rpy="0 0 0"/>
             <geometry>
-                <box size="0.22 0.14 0.06"/>
+                <box size="0.22 0.10 0.06"/>
             </geometry>
         </collision>
@@ -55,4 +55,5 @@
         <origin xyz="-0.035 0.065 0.03" rpy="0 0 0"/>
         <axis xyz="0 1 0"/>
+        <limit effort="100.0" velocity="100.0"/>
     </joint>
     <link name="left_front_wheel">
@@ -80,4 +81,5 @@
         <origin xyz="0.073 0.065 0.03" rpy="0 0 0"/>
         <axis xyz="0 1 0"/>
+        <limit effort="100.0" velocity="100.0"/>
     </joint>
     <link name="right_rear_wheel">
@@ -105,4 +107,5 @@
         <origin xyz="-0.035 -0.09 0.03" rpy="0 0 0"/>
         <axis xyz="0 1 0"/>
+        <limit effort="100.0" velocity="100.0"/>
     </joint>
     <link name="right_front_wheel">
@@ -130,4 +133,5 @@
         <origin xyz="0.073 -0.09 0.03" rpy="0 0 0"/>
         <axis xyz="0 1 0"/>
+        <limit effort="100.0" velocity="100.0"/>
     </joint>
     <link name="camera_link">
